File: analog.sch (KiCad schematic (older format))
At the start: 102 parts, among them J10 Conn_01x02_Female, J11 Conn_01x02_Male, J12 Conn_01x02_Male, J13 Conn_01x02_Female, J14 Conn_01x02_Male, J15 Conn_01x02_Female, J4 Conn_01x04_Male, J5 Conn_01x04_Male, J8 Conn_01x02_Male, J9 Conn_01x02_Female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

Commit message: Updated board size to fit in housing
Parts:
- U17, U18: footprint MAX3806GTCT:21-0136I_T1233-3 -> maximsmd:QFN-12-1EP_4x4mm_P0.8mm
Changed lines of the file:
@@
 F 0 "U17" H 2450 3400 50  0000 C CNN
 F 1 "MAX1932" H 2750 2800 50  0000 C CNB
-F 2 "MAX3806GTCT:21-0136I_T1233-3" H 2400 3450 50  0001 C CNN
+F 2 "maximsmd:QFN-12-1EP_4x4mm_P0.8mm" H 2400 3450 50  0001 C CNN
 F 3 "" H 2400 3450 50  0001 C CNN
 	1    2750 2700
@@
 F 0 "U18" H 2450 6500 50  0000 C CNN
 F 1 "MAX1932" H 2750 5900 50  0000 C CNB
-F 2 "MAX3806GTCT:21-0136I_T1233-3" H 2400 6550 50  0001 C CNN
+F 2 "maximsmd:QFN-12-1EP_4x4mm_P0.8mm" H 2400 6550 50  0001 C CNN
 F 3 "" H 2400 6550 50  0001 C CNN
 	1    2750 5800
